File: reform2-motherboard-pcb/reform2-hdmi.sch (KiCad schematic (older format))
At the start: 16 parts, among them J4 HDMI_A, U22 TPD12S521

Commit message: motherboard: add the split-up and cleaned up schematics that were made for the book
Parts:
- J4: symbol Connector:HDMI_A -> reform2-motherboard-rescue:HDMI_A-nologo
Other:
- note added: "HDMI\nConnector"
- note added: "Port\nProtection"
- moved on the sheet: C27, C28, C29, C30, D14, R161, R192, R197, R43, R44, R45, R46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
