File: reform2-motherboard-pcb/reform2-motherboard.sch (KiCad schematic (older format))
At the start: 44 parts, among them J15 Conn_01x33, J18 Conn_01x03_Male, J19 JTAG, J20 Conn_01x03_Male, SW3 SW_DIP_x01, SW5 SW_DIP_x04, SW6 SW_Push, U1 Nitrogen8M

Commit message: motherboard: add the split-up and cleaned up schematics that were made for the book
Parts:
- H1: DNP y -> (none); Manufacturer (none) -> Wurth; Manufacturer_No (none) -> 9774020243R
- H22, H24, H25, H27: Manufacturer_No 9774010243 -> 9774025243R
- U1: value Nitrogen8M -> Nitrogen8M_SOM; symbol reform2:Nitrogen8M -> reform2-motherboard-rescue:Nitrogen8M-reform2
Connections:
- net labels added: IMX_FBOOT
- net labels removed: IMX_PWM4
- wire segments 207 -> 259
Other:
- note added: "AUX UART (SER2)"
- note added: "Boot UART (SER1)"
- note added: "Refclk input \n(PAD_CLK) \nfor PCIe2"
- note added: "User defined switch (XSW)"
- note added: "i.MX8M internal \noscillator output \nfor PCIe1"
- note removed: "AUX UART"
- note removed: "Boot UART"
- note removed: "NOTE: optimize bead values?\nhttps://www.allaboutcircuits.com/technical-articles/choosing-and-using-ferrite-beads/\nhttps://www.we-online.com/catalog/datasheet/74279265.pdf\nsamsung CIS21J121NE"
- note removed: "This is a i.MX8M internal oscillator output for PCIe1"
- note removed: "This is refclk input (PAD_CLK) for PCIe2"
- moved on the sheet: H1, H10, H11, H12, H13, H14, H15, H2, H22, H24, H25, H27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
