File: reform2-motherboard-pcb/reform2-power.sch (KiCad schematic (older format))
At the start: 202 parts, among them J1 Jack-DC, J13 BATCON1, J2 BATCON2, J22 LPC_IO, J23 KDBSYSCTL, J8 USB_B_Micro, Q1 Si7850DP, Q10 PMV50EPEAR, Q11 PMV50EPEAR, Q12 PMV50EPEAR, Q13 PMV50ENEAR, Q14 PMV50ENEAR, Q15 Si7850DP, Q17 Si7850DP, Q18 Si7461DP, Q2 Si7850DP, Q3 Si7461DP, Q4 PMV50ENEAR, Q5 PMV50EPEAR, Q6 PMV50EPEAR, Q7 PMV50EPEAR, Q8 PMV50EPEAR, Q9 PMV50EPEAR, SW1 SW_DIP_x01, SW2 SW_Push, U12 LM2677SX-3.3, U13 TLV62568DBV, U14 LMR16006YQ3, U17 TLV1117-18, U18 LPC11U24FBD48-301, U19 TLV62568DBV, U2 LTC4020EUHFPBF, U4 LTC6803-4, U5 PCF8523T, U6 INA260, U7 LM2677SX-5, Y2 12MHz, Y4 32.768 kHz

Commit message: motherboard: add the split-up and cleaned up schematics that were made for the book
Parts:
- removed BT1: CR1220, Battery:BatteryHolder_Keystone_3000_1x12mm, symbol Device:Battery_Cell
- removed C121: 47uF, Capacitor_SMD:C_0603_1608Metric, symbol Device:C_Small
- removed C128, C148: 10nF, Capacitor_SMD:C_0603_1608Metric, symbol Device:C_Small
- removed C129, C130, C145, C146: 1uF, Capacitor_SMD:C_0603_1608Metric, symbol Device:C_Small
- removed C140, C49, C50: 0.1uF, Capacitor_SMD:C_0603_1608Metric, symbol Device:C_Small
- removed C16, C17: 100uF, Capacitor_SMD:CP_Elec_8x10, symbol Device:CP_Small
- removed C18, C19: 220uF, Capacitor_SMD:CP_Elec_8x10, symbol Device:CP_Small
- removed C3: 0.33uF, Capacitor_SMD:C_0603_1608Metric, symbol Device:C_Small
- removed C33, C35: 4.7uF, Capacitor_SMD:C_0603_1608Metric, symbol Device:C_Small
- removed C34, C37, C46, C47: 10uF, Capacitor_SMD:C_0603_1608Metric, symbol Device:C_Small
- removed C36, C38: 6.8pF, Capacitor_SMD:C_0603_1608Metric, symbol Device:C_Small
- removed C48, C51: 18pF, Capacitor_SMD:C_0603_1608Metric, symbol reform2-motherboard-rescue:C_Small-reform-motherboard-rescue
- removed C82: 2.2uF, Capacitor_SMD:C_0603_1608Metric, symbol Device:C_Small
- removed D11: LED3V, LED_SMD:LED_0603_1608Metric, symbol Device:LED_Small_ALT
- removed D12: LED5V, LED_SMD:LED_0603_1608Metric, symbol Device:LED_Small_ALT
- removed D20, D21: SK54A-LTP, Diode_SMD:D_SMA, symbol Diode:1N5821
- removed D3: SBR0560S1, Diode_SMD:D_SOD-123, symbol Device:D_Schottky_Small_ALT
- removed J22: LPC_IO, Connector_PinHeader_2.54mm:PinHeader_2x08_P2.54mm_Vertical, symbol Connector_Generic:Conn_02x08_Odd_Even
- removed J23: KDBSYSCTL, Connector_JST:JST_PH_B4B-PH-K_1x04_P2.00mm_Vertical, symbol Connector:Conn_01x04_Male
- removed J8: USB_B_Micro, footprints:WE_629105136821, symbol Connector:USB_B_Micro
- removed L3, L4: 68uH, Inductor_SMD:L_Bourns_SRR1210A, symbol Device:L
- removed L5: 10uH, Inductor_SMD:L_1210_3225Metric, symbol Device:L
- removed L6, L7: 2.2uH, Inductor_SMD:L_1210_3225Metric, symbol Device:L_Small
- removed Q13, Q14: PMV50ENEAR, Package_TO_SOT_SMD:SOT-23, symbol Transistor_FET:2N7002E
- removed R1, R100, R124, R125, R126, R127, R137, R157, R185, R186, R194, R73, R74, R75, R76, R98: 0, Resistor_SMD:R_0603_1608Metric, symbol Device:R_Small
- removed R128: 10k, Resistor_SMD:R_0603_1608Metric, symbol Device:R_Small
- removed R164, R33: 1k, Resistor_SMD:R_0603_1608Metric, symbol Device:R_Small
- removed R178, R179, R181, R188, R189, R88, R89: 100k, Resistor_SMD:R_0603_1608Metric, symbol Device:R_Small
- removed R180: 150k, Resistor_SMD:R_0603_1608Metric, symbol Device:R_Small
- removed R195, R71: 1.5k, Resistor_SMD:R_0603_1608Metric, symbol Device:R_Small
- removed R68, R69: 4.7k, Resistor_SMD:R_0603_1608Metric, symbol Device:R_Small
- removed R70, R72: 33, Resistor_SMD:R_0603_1608Metric, symbol Device:R_Small
- removed SW1: SW_DIP_x01, Button_Switch_SMD:SW_DIP_SPSTx01_Slide_Omron_A6S-110x_W8.9mm_P2.54mm, symbol Switch:SW_DIP_x01
- removed SW2: SW_Push, footprints:UK-B0206-G3.8-250-JZ, symbol Switch:SW_Push
- removed U12: LM2677SX-3.3, Package_TO_SOT_SMD:TO-263-7_TabPin8, symbol reform2:LM2677-3.3
- removed U13, U19: TLV62568DBV, Package_TO_SOT_SMD:SOT-23-5, symbol Regulator_Switching:TLV62568DBV
- removed U14: LMR16006YQ3, Package_TO_SOT_SMD:TSOT-23-6, symbol Regulator_Switching:LM2841X
- removed U17: TLV1117-18, Package_TO_SOT_SMD:SOT-223, symbol Regulator_Linear:TLV1117-18
- removed U18: LPC11U24FBD48-301, Package_QFP:LQFP-48_7x7mm_P0.5mm, symbol MCU_NXP_LPC:LPC11U24FBD48-301
- removed U5: PCF8523T, Package_SO:SOIC-8_3.9x4.9mm_P1.27mm, symbol Timer_RTC:PCF8523T
- removed U7: LM2677SX-5, Package_TO_SOT_SMD:TO-263-7_TabPin8, symbol reform2:LM2677-3.3
- removed Y2: 12MHz, Crystal:Crystal_SMD_Abracon_ABM8G-4Pin_3.2x2.5mm, symbol Device:Crystal_GND24_Small
- removed Y4: 32.768 kHz, Crystal:Crystal_SMD_3215-2Pin_3.2x1.5mm, symbol Device:Crystal_Small
Connections:
- net labels added: CHGBAT, VIN
- net labels removed: +1V2, +1V5, +1V8, +3V3, +5V, 3V3_PWR_AUX, AUX_PWR_EN, DAC_SCL, DAC_SDA, IMX_RESETn, IMX_RTC_IRQ, IMX_WAKE, LPCUD_N, LPCUD_P, LPC_AD5, LPC_AD7, LPC_MISO, LPC_MISO0, LPC_MISO1a, LPC_MISO1b, LPC_MOSI, LPC_MOSI0, LPC_MOSI1a, LPC_MOSI1b, LPC_PIO0_20, LPC_PIO1_16, LPC_PIO1_24, LPC_PIO1_25, LPC_PIO1_31, LPC_RXDa, LPC_RXDb, LPC_RXDc, LPC_SCK, LPC_SCK0a, LPC_SCK0b, LPC_SCK1a, LPC_SCK1b, LPC_SCL, LPC_SCLKa, LPC_SCLKc, LPC_SDA, LPC_SS0, LPC_SSEL0, LPC_SSEL1, LPC_SWDIO, LPC_TDI, LPC_TDO, LPC_TMS, LPC_TXDa, LPC_TXDb, LPC_TXDc, LPC_UART2_RX, LPC_UART2_TX, LPC_UFTOGG, LPC_UVBUS, LPC_~CTS, LPC_~DTR, LPC_~RESET, LPC_~TRST, LPC_~USBCON, PCIE1_PWR_EN, USB_PWR_EN
- wire segments 730 -> 434
- no-connect marks 8 -> 5
Other:
- note added: "12-24VDC\nInput"
- note added: "Balancer"
- note added: "Battery current\nand voltage monitor"
- note added: "Charge current\nlimit control\n(toggles no charge\n/no limit)"
- note added: "Charger/\nBooster"
- note added: "Close to PVIN"
- note added: "Inrush Current\nLimiter by Zoé"
- note added: "LiFePO4\nBattery\nStack"
- note added: "Oscillator freq\ncontrol. 100k = 250kHz"
- note added: "Status LEDs"
- note removed: "12-24VDC"
- note removed: "1A"
- note removed: "BALANCER"
- note removed: "EN_1V2!"
- note removed: "EN_3V3"
- note removed: "EN_3V3!"
- note removed: "EN_5V"
- note removed: "EN_5V!"
- note removed: "I2C lines pulled up\nby SYS 3v3 power\nnear DAC"
- note removed: "Keyboard System Control Port"
- note removed: "LIFEPO4 \nBATTERY \nSTACK"
- note removed: "Main system power\nconverters, enabled\nby LPC"
- note removed: "Powered by \nmain batteries\nin standby"
- note removed: "Powered by coin\ncell when batteries\nremoved"
- note removed: "Realtime Clock"
- note removed: "These values are\ncopied from the\ndatasheet and should\nbe verified with a VNA"
- note removed: "Up to 5A @ 3.3V"
- note removed: "Up to 5A @ 5V"
- note removed: "VCCIO supply for DSI + SD"
- note removed: "battery current\nand voltage monitor"
- note removed: "charge current\nlimit control\n(toggles no charge\n/no limit)"
- note removed: "close to PVIN"
- note removed: "inrush current\nlimiter, thanks zoé"
- note removed: "oscillator freq\ncontrol. 100k = 250kHz"
- note removed: "standby always-on\npower rail"
- note removed: "up to 1A (peak)\n375mA normal \nfrom mPCIe"
- note removed: "up to 40mA consumed \nby DSI bridge and\nSD card level shifter"
- note removed: "up to 70mA consumed \nby DSI bridge"
- note removed: "up to 780mA (!)\nconsumed by USB hub"
- moved on the sheet: C1, C10, C11, C12, C122, C125, C13, C14, C149, C15, C160, C161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
