File: reform2-motherboard-pcb/reform2-usb.sch (KiCad schematic (older format))
At the start: 86 parts, among them J14 USB_INT2, J17 USB3_A, J5 USB3_A, J6 USB3_A, J9 USB_INT1, U15 TPS2561, U16 TPS2561, U21 SP3012-06UTG, U24 AP22815, U25 SP3012-06UTG, U26 SP3012-06UTG, U27 AP22815, U9 TUSB8041IPAPRQ1, Y1 24MHz

Commit message: motherboard: add the split-up and cleaned up schematics that were made for the book
Parts:
- removed C164, C167: 10uF, Capacitor_SMD:C_0603_1608Metric, symbol Device:C_Small
- removed C66, C73: 0.1uF, Capacitor_SMD:C_0603_1608Metric, symbol Device:C_Small
- removed D15: SD0603S040S0R2, Diode_SMD:D_0603_1608Metric_Castellated, symbol Device:D_Schottky_Small
- removed R2, R83: 10k, Resistor_SMD:R_0603_1608Metric, symbol Device:R_Small
- removed R81, R84, R85, R86: 100k, Resistor_SMD:R_0603_1608Metric, symbol Device:R_Small
- removed R87, R99: 24.9k, Resistor_SMD:R_0603_1608Metric, symbol Device:R_Small
- removed U15, U16: TPS2561, Package_SON:VSON-10-1EP_3x3mm_P0.5mm_EP1.65x2.4mm_ThermalVias, symbol Interface_USB:TPS2561
- removed U24, U27: AP22815, footprints:TSOT-25, symbol reform2:AP22815
- J17, J5, J6: symbol Connector:USB3_A -> reform2-motherboard-rescue:USB3_A-Connector
Connections:
- net labels removed: +3V3, +5V, AUX_PWR_EN, USB_PWR_EN
- wire segments 301 -> 240
Other:
- note added: "Protection"
- note added: "USB Hub"
- note added: "Up to 780mA load!"
- note removed: "TODO: consider internal USB3"
- note removed: "up to 780mA load!"
- moved on the sheet: C20, C21, C39, C40, C41, C42, C43, C63, C67, C68, C69, C70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
