File: reform2-trackball-sensor-pcb/reform2-trackball-sensor.kicad_pcb (KiCad board)
At the start: 2 copper layers, 23.8 x 17.8 mm, 10 parts, among them J1 Conn_01x06_Male, U1 PAT9125EL

Commit message: reform2: update PCBs incl. badges to production revs, add keyboard lettering, misc docs
Parts:
- H8: footprint footprints:mnt-minilogo -> footprints-sensor:reform2-trackball-sensor-badge
- moved H8 6.75 mm to (155.2, 81.6), turned to 0 degrees
