File: reform2-motherboard25-pcb/reform2-sd.kicad_sch (KiCad schematic)
At the start: 13 parts, among them J3 SD_Card, U28 SN74AVC1T45, U8 TXS0108EPW

Commit message: motherboard 2.5 snapshot: fully routed and cleaned up
Parts:
- C138, C168, C169, C56, C57: Distributor Mouser -> (none)
Changed lines of the file:
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@@
       (effects (font (size 1.27 1.27)) hide)
     )
-    (property "Distributor" "Mouser" (id 7) (at 119.38 81.28 0)
+    (property "Distributor" "" (id 7) (at 119.38 81.28 0)
       (effects (font (size 1.27 1.27)) hide)
     )
@@
       (effects (font (size 1.27 1.27)) hide)
     )
-    (property "Distributor" "Mouser" (id 7) (at 93.98 67.31 0)
+    (property "Distributor" "" (id 7) (at 93.98 67.31 0)
       (effects (font (size 1.27 1.27)) hide)
     )
@@
       (effects (font (size 1.27 1.27)) hide)
     )
-    (property "Distributor" "Mouser" (id 7) (at 146.05 80.01 0)
+    (property "Distributor" "" (id 7) (at 146.05 80.01 0)
       (effects (font (size 1.27 1.27)) hide)
     )
@@
       (effects (font (size 1.27 1.27)) hide)
     )
-    (property "Distributor" "Mouser" (id 7) (at 130.81 143.51 0)
+    (property "Distributor" "" (id 7) (at 130.81 143.51 0)
       (effects (font (size 1.27 1.27)) hide)
     )
@@
       (effects (font (size 1.27 1.27)) hide)
     )
-    (property "Distributor" "Mouser" (id 7) (at 67.31 143.51 0)
-      (effects (font (size 1.27 1.27)) hide)
-    )
+    (property "Distributor" "" (id 7) (at 67.31 143.51 0)
+      (effects (font (size 1.27 1.27)) hide)
+    )
