File: reform2-motherboard25-pcb/reform2-audio.kicad_sch (KiCad schematic)
At the start: 53 parts, among them J16 LINE_IN, J21 Conn_01x04, J7 SJ-43516-SMT, U3 WM8960

Commit message: motherboard 2.5 snapshot: fully routed and cleaned up
Parts:
- C142, C143, C144, C154, C156, C158, C165, C166: Distributor Mouser -> (none)
Changed lines of the file:
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@@
       (effects (font (size 1.27 1.27)) hide)
     )
-    (property "Distributor" "Mouser" (id 7) (at 106.68 68.58 0)
+    (property "Distributor" "" (id 7) (at 106.68 68.58 0)
       (effects (font (size 1.27 1.27)) hide)
     )
@@
       (effects (font (size 1.27 1.27)) hide)
     )
-    (property "Distributor" "Mouser" (id 7) (at 106.68 74.93 0)
+    (property "Distributor" "" (id 7) (at 106.68 74.93 0)
       (effects (font (size 1.27 1.27)) hide)
     )
@@
       (effects (font (size 1.27 1.27)) hide)
     )
-    (property "Distributor" "Mouser" (id 7) (at 170.18 147.32 0)
+    (property "Distributor" "" (id 7) (at 170.18 147.32 0)
       (effects (font (size 1.27 1.27)) hide)
     )
@@
       (effects (font (size 1.27 1.27)) hide)
     )
-    (property "Distributor" "Mouser" (id 7) (at 113.03 119.38 0)
+    (property "Distributor" "" (id 7) (at 113.03 119.38 0)
       (effects (font (size 1.27 1.27)) hide)
     )
@@
       (effects (font (size 1.27 1.27)) hide)
     )
-    (property "Distributor" "Mouser" (id 7) (at 173.99 113.03 0)
+    (property "Distributor" "" (id 7) (at 173.99 113.03 0)
       (effects (font (size 1.27 1.27)) hide)
     )
@@
       (effects (font (size 1.27 1.27)) hide)
     )
-    (property "Distributor" "Mouser" (id 7) (at 176.53 119.38 0)
+    (property "Distributor" "" (id 7) (at 176.53 119.38 0)
       (effects (font (size 1.27 1.27)) hide)
     )
@@
       (effects (font (size 1.27 1.27)) hide)
     )
-    (property "Distributor" "Mouser" (id 7) (at 179.07 125.73 0)
+    (property "Distributor" "" (id 7) (at 179.07 125.73 0)
       (effects (font (size 1.27 1.27)) hide)
     )
@@
       (effects (font (size 1.27 1.27)) hide)
     )
-    (property "Distributor" "Mouser" (id 7) (at 181.61 132.08 0)
-      (effects (font (size 1.27 1.27)) hide)
-    )
+    (property "Distributor" "" (id 7) (at 181.61 132.08 0)
+      (effects (font (size 1.27 1.27)) hide)
+    )

Commit message: motherboard25: r-1 snapshot, ordered for test bringup
Parts:
- C127, C147: Checked (none) -> y
- J16: Manufacturer (none) -> Generic; Manufacturer_No (none) -> 3P 2mm pitch THT header
Changed lines of the file:
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@@
       (effects (font (size 1.27 1.27)) hide)
     )
-    (property "Checked" "" (id 6) (at 160.02 90.17 0)
+    (property "Checked" "y" (id 6) (at 160.02 90.17 0)
       (effects (font (size 1.27 1.27)) hide)
     )
@@
       (effects (font (size 1.27 1.27)) hide)
     )
-    (property "Checked" "" (id 6) (at 160.02 97.79 0)
+    (property "Checked" "y" (id 6) (at 160.02 97.79 0)
       (effects (font (size 1.27 1.27)) hide)
     )
@@
       (effects (font (size 1.27 1.27)) hide)
     )
+    (property "Manufacturer" "Generic" (id 6) (at 140.97 46.99 0)
+      (effects (font (size 1.27 1.27)) hide)
+    )
+    (property "Manufacturer_No" "3P 2mm pitch THT header" (id 7) (at 140.97 46.99 0)
+      (effects (font (size 1.27 1.27)) hide)
+    )
