File: reform2-motherboard25-pcb/reform2-display.kicad_sch (KiCad schematic)
At the start: 38 parts, among them J24 EDP_HEADER, U10 SN65DSI86IPAPQ1

Commit message: motherboard 2.5 snapshot: fully routed and cleaned up
Parts:
- C101, C103, C105, C106, C107, C108, C109, C110, C113, C115, C118, C135, C136: Distributor Mouser -> (none)
- J24: Manufacturer Molex -> Molex / Würth; Manufacturer_No 87758-3016 -> 87758-3016 / 687133149022
Changed lines of the file:
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@@
       (effects (font (size 1.27 1.27)) hide)
     )
-    (property "Manufacturer" "Molex" (id 4) (at 233.68 58.42 0)
-      (effects (font (size 1.27 1.27)) hide)
-    )
-    (property "Manufacturer_No" "87758-3016" (id 5) (at 233.68 58.42 0)
+    (property "Manufacturer" "Molex / Würth" (id 4) (at 233.68 58.42 0)
+      (effects (font (size 1.27 1.27)) hide)
+    )
+    (property "Manufacturer_No" "87758-3016 / 687133149022" (id 5) (at 233.68 58.42 0)
       (effects (font (size 1.27 1.27)) hide)
     )
@@
       (effects (font (size 1.27 1.27)) hide)
     )
-    (property "Distributor" "Mouser" (id 7) (at 64.77 36.83 0)
+    (property "Distributor" "" (id 7) (at 64.77 36.83 0)
       (effects (font (size 1.27 1.27)) hide)
     )
@@
       (effects (font (size 1.27 1.27)) hide)
     )
-    (property "Distributor" "Mouser" (id 7) (at 86.36 36.83 0)
+    (property "Distributor" "" (id 7) (at 86.36 36.83 0)
       (effects (font (size 1.27 1.27)) hide)
     )
@@
       (effects (font (size 1.27 1.27)) hide)
     )
-    (property "Distributor" "Mouser" (id 7) (at 148.59 115.57 0)
+    (property "Distributor" "" (id 7) (at 148.59 115.57 0)
       (effects (font (size 1.27 1.27)) hide)
     )
@@
       (effects (font (size 1.27 1.27)) hide)
     )
-    (property "Distributor" "Mouser" (id 7) (at 170.18 115.57 0)
+    (property "Distributor" "" (id 7) (at 170.18 115.57 0)
       (effects (font (size 1.27 1.27)) hide)
     )
@@
       (effects (font (size 1.27 1.27)) hide)
     )
-    (property "Distributor" "Mouser" (id 7) (at 157.48 138.43 0)
+    (property "Distributor" "" (id 7) (at 157.48 138.43 0)
       (effects (font (size 1.27 1.27)) hide)
     )
@@
       (effects (font (size 1.27 1.27)) hide)
     )
-    (property "Distributor" "Mouser" (id 7) (at 142.24 69.85 0)
+    (property "Distributor" "" (id 7) (at 142.24 69.85 0)
       (effects (font (size 1.27 1.27)) hide)
     )
@@
       (effects (font (size 1.27 1.27)) hide)
     )
-    (property "Distributor" "Mouser" (id 7) (at 148.59 72.39 0)
+    (property "Distributor" "" (id 7) (at 148.59 72.39 0)
       (effects (font (size 1.27 1.27)) hide)
     )
@@
       (effects (font (size 1.27 1.27)) hide)
     )
-    (property "Distributor" "Mouser" (id 7) (at 142.24 77.47 0)
+    (property "Distributor" "" (id 7) (at 142.24 77.47 0)
       (effects (font (size 1.27 1.27)) hide)
     )
@@
       (effects (font (size 1.27 1.27)) hide)
     )
-    (property "Distributor" "Mouser" (id 7) (at 148.59 80.01 0)
+    (property "Distributor" "" (id 7) (at 148.59 80.01 0)
       (effects (font (size 1.27 1.27)) hide)
     )
@@
       (effects (font (size 1.27 1.27)) hide)
     )
-    (property "Distributor" "Mouser" (id 7) (at 142.24 85.09 0)
+    (property "Distributor" "" (id 7) (at 142.24 85.09 0)
       (effects (font (size 1.27 1.27)) hide)
     )
@@
       (effects (font (size 1.27 1.27)) hide)
     )
-    (property "Distributor" "Mouser" (id 7) (at 148.59 87.63 0)
+    (property "Distributor" "" (id 7) (at 148.59 87.63 0)
       (effects (font (size 1.27 1.27)) hide)
     )
@@
       (effects (font (size 1.27 1.27)) hide)
     )
-    (property "Distributor" "Mouser" (id 7) (at 243.84 147.32 0)
+    (property "Distributor" "" (id 7) (at 243.84 147.32 0)
       (effects (font (size 1.27 1.27)) hide)
     )
@@
       (effects (font (size 1.27 1.27)) hide)
     )
-    (property "Distributor" "Mouser" (id 7) (at 243.84 119.38 0)
-      (effects (font (size 1.27 1.27)) hide)
-    )
+    (property "Distributor" "" (id 7) (at 243.84 119.38 0)
+      (effects (font (size 1.27 1.27)) hide)
+    )

Commit message: motherboard25: r-1 snapshot, ordered for test bringup
Connections:
- net at C100.1, C101.1, C102.1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: now also U10.14 (VCCA)
Changed lines of the file:
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@@
   (junction (at 109.22 44.45) (diameter 0) (color 0 0 0 0)
+  )
+  (junction (at 104.14 44.45) (diameter 0) (color 0 0 0 0)
   )
   (junction (at 129.54 118.11) (diameter 0) (color 0 0 0 0)
@@
     (stroke (width 0) (type default) (color 0 0 0 0))
   )
+  (wire (pts (xy 104.14 44.45) (xy 106.68 44.45))
+    (stroke (width 0) (type default) (color 0 0 0 0))
+  )
   (wire (pts (xy 55.88 39.37) (xy 45.72 39.37))
     (stroke (width 0) (type default) (color 0 0 0 0))
@@
     (stroke (width 0) (type default) (color 0 0 0 0))
   )
+  (wire (pts (xy 104.14 44.45) (xy 104.14 49.53))
+    (stroke (width 0) (type default) (color 0 0 0 0))
+  )
   (wire (pts (xy 54.61 133.35) (xy 55.88 133.35))
     (stroke (width 0) (type default) (color 0 0 0 0))
   )
-  (wire (pts (xy 101.6 44.45) (xy 106.68 44.45))
+  (wire (pts (xy 101.6 44.45) (xy 104.14 44.45))
     (stroke (width 0) (type default) (color 0 0 0 0))
   )
@@
       (effects (font (size 1.27 1.27)) (justify left bottom) hide)
     )
-    (property "Datasheet" "http://www.ti.com/lit/ds/symlink/sn65dsi86-q1.pdf" (id 3) (at 102.87 95.25 0)
+    (property "Datasheet" "http://www.ti.com/lit/ds/symlink/sn65dsi86-q1.pdf" (id 3) (at 100.33 34.29 0)
       (effects (font (size 1.27 1.27)) (justify left bottom) hide)
     )
-    (property "Manufacturer" "Texas Instruments" (id 4) (at 102.87 95.25 0)
-      (effects (font (size 1.27 1.27)) hide)
-    )
-    (property "Manufacturer_No" "SN65DSI86IPAPQ1" (id 5) (at 102.87 95.25 0)
+    (property "Manufacturer" "Texas Instruments" (id 4) (at 104.14 99.06 0)
+      (effects (font (size 1.27 1.27)) hide)
+    )
+    (property "Manufacturer_No" "SN65DSI86IPAPQ1" (id 5) (at 104.14 90.17 0)
       (effects (font (size 1.27 1.27)) hide)
     )
@@
       (effects (font (size 1.27 1.27)) hide)
     )
-    (property "Distributor" "Mouser" (id 7) (at 102.87 95.25 0)
+    (property "Distributor" "Mouser" (id 7) (at 104.14 101.6 0)
       (effects (font (size 1.27 1.27)) hide)
     )
@@
     (pin "12")
     (pin "13")
+    (pin "14")
     (pin "15")
     (pin "16")
