File: reform2-motherboard25-pcb/reform2-eth.kicad_sch (KiCad schematic)
At the start: 9 parts, among them P1 J0G-0003NL

Commit message: motherboard 2.5 snapshot: fully routed and cleaned up
Parts:
- C22, C23, C24, C25, C26: Distributor Mouser -> (none)
Changed lines of the file:
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@@
       (effects (font (size 1.27 1.27)) hide)
     )
-    (property "Distributor" "Mouser" (id 7) (at 83.82 130.81 0)
+    (property "Distributor" "" (id 7) (at 83.82 130.81 0)
       (effects (font (size 1.27 1.27)) hide)
     )
@@
       (effects (font (size 1.27 1.27)) hide)
     )
-    (property "Distributor" "Mouser" (id 7) (at 104.14 55.88 0)
+    (property "Distributor" "" (id 7) (at 104.14 55.88 0)
       (effects (font (size 1.27 1.27)) hide)
     )
@@
       (effects (font (size 1.27 1.27)) hide)
     )
-    (property "Distributor" "Mouser" (id 7) (at 104.14 76.2 0)
+    (property "Distributor" "" (id 7) (at 104.14 76.2 0)
       (effects (font (size 1.27 1.27)) hide)
     )
@@
       (effects (font (size 1.27 1.27)) hide)
     )
-    (property "Distributor" "Mouser" (id 7) (at 104.14 96.52 0)
+    (property "Distributor" "" (id 7) (at 104.14 96.52 0)
       (effects (font (size 1.27 1.27)) hide)
     )
@@
       (effects (font (size 1.27 1.27)) hide)
     )
-    (property "Distributor" "Mouser" (id 7) (at 104.14 116.84 0)
+    (property "Distributor" "" (id 7) (at 104.14 116.84 0)
       (effects (font (size 1.27 1.27)) hide)
     )

Commit message: motherboard25: r-1 snapshot, ordered for test bringup
Parts:
- P1: Availability Good -> (none)
Changed lines of the file:
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@@
-      (effects (font (size 1.27 1.27)) (justify left bottom) hide)
-    )
-    (property "Availability" "Good" (id 4) (at 147.32 96.52 0)
       (effects (font (size 1.27 1.27)) (justify left bottom) hide)
     )
