File: reform2-motherboard25-pcb/reform2-hdmi.kicad_sch (KiCad schematic)
At the start: 16 parts, among them J4 HDMI_A, U22 TPD12S521

Commit message: motherboard 2.5 snapshot: fully routed and cleaned up
Parts:
- C27, C28, C29, C30, R161, R45: Distributor Mouser -> (none)
Changed lines of the file:
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@@
       (effects (font (size 1.27 1.27)) hide)
     )
-    (property "Distributor" "Mouser" (id 7) (at 186.69 140.97 0)
+    (property "Distributor" "" (id 7) (at 186.69 140.97 0)
       (effects (font (size 1.27 1.27)) hide)
     )
@@
       (effects (font (size 1.27 1.27)) hide)
     )
-    (property "Distributor" "Mouser" (id 7) (at 182.88 35.56 0)
+    (property "Distributor" "" (id 7) (at 182.88 35.56 0)
       (effects (font (size 1.27 1.27)) hide)
     )
@@
       (effects (font (size 1.27 1.27)) hide)
     )
-    (property "Distributor" "Mouser" (id 7) (at 162.56 104.14 0)
+    (property "Distributor" "" (id 7) (at 162.56 104.14 0)
       (effects (font (size 1.27 1.27)) hide)
     )
@@
       (effects (font (size 1.27 1.27)) hide)
     )
-    (property "Distributor" "Mouser" (id 7) (at 151.13 101.6 0)
+    (property "Distributor" "" (id 7) (at 151.13 101.6 0)
       (effects (font (size 1.27 1.27)) hide)
     )
@@
       (effects (font (size 1.27 1.27)) hide)
     )
-    (property "Distributor" "Mouser" (id 7) (at 147.32 114.3 0)
+    (property "Distributor" "" (id 7) (at 147.32 114.3 0)
       (effects (font (size 1.27 1.27)) hide)
     )
@@
       (effects (font (size 1.27 1.27)) hide)
     )
-    (property "Distributor" "Mouser" (id 5) (at 153.67 104.14 0)
-      (effects (font (size 1.27 1.27)) hide)
-    )
+    (property "Distributor" "" (id 5) (at 153.67 104.14 0)
+      (effects (font (size 1.27 1.27)) hide)
+    )

Commit message: motherboard25: r-1 snapshot, ordered for test bringup
Parts:
- R161, R45: Distributor (none) -> Mouser
Changed lines of the file:
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@@
       (effects (font (size 1.27 1.27)) hide)
     )
-    (property "Distributor" "" (id 7) (at 186.69 140.97 0)
+    (property "Distributor" "Mouser" (id 7) (at 186.69 140.97 0)
       (effects (font (size 1.27 1.27)) hide)
     )
@@
       (effects (font (size 1.27 1.27)) hide)
     )
-    (property "Distributor" "" (id 5) (at 153.67 104.14 0)
-      (effects (font (size 1.27 1.27)) hide)
-    )
+    (property "Distributor" "Mouser" (id 5) (at 153.67 104.14 0)
+      (effects (font (size 1.27 1.27)) hide)
+    )
