File: reform2-motherboard25-pcb/reform2-lpc.kicad_sch (KiCad schematic)
At the start: 34 parts, among them J22 LPC_IO, J23 KDBSYSCTL, J8 USB_C_Receptacle_USB2.0, SW1 SW_DIP_x01, SW2 SW_Push, U18 LPC11U24FBD48-301, U5 PCF8523T, Y2 12MHz, Y4 32.768 kHz

Commit message: motherboard 2.5 snapshot: fully routed and cleaned up
Parts:
- C140, C49, C50, R128: Distributor Mouser -> (none)
Changed lines of the file:
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@@
       (effects (font (size 1.27 1.27)) hide)
     )
-    (property "Distributor" "Mouser" (id 7) (at 162.56 50.8 0)
+    (property "Distributor" "" (id 7) (at 162.56 50.8 0)
       (effects (font (size 1.27 1.27)) hide)
     )
@@
       (effects (font (size 1.27 1.27)) hide)
     )
-    (property "Distributor" "Mouser" (id 7) (at 172.72 50.8 0)
+    (property "Distributor" "" (id 7) (at 172.72 50.8 0)
       (effects (font (size 1.27 1.27)) hide)
     )
@@
       (effects (font (size 1.27 1.27)) hide)
     )
-    (property "Distributor" "Mouser" (id 7) (at 191.77 73.66 0)
+    (property "Distributor" "" (id 7) (at 191.77 73.66 0)
       (effects (font (size 1.27 1.27)) hide)
     )
@@
       (effects (font (size 1.27 1.27)) hide)
     )
-    (property "Distributor" "Mouser" (id 7) (at 44.45 160.02 0)
-      (effects (font (size 1.27 1.27)) hide)
-    )
+    (property "Distributor" "" (id 7) (at 44.45 160.02 0)
+      (effects (font (size 1.27 1.27)) hide)
+    )

Commit message: motherboard25: r-1 snapshot, ordered for test bringup
Parts:
- C48, C51: LCSC (none) -> C107040
- J8: Checked (none) -> y; Distributor (none) -> LCSC; LCSC (none) -> C165948; Manufacturer (none) -> Korean Hroparts; Manufacturer_No (none) -> TYPE-C-31-M-12
- R128: Distributor (none) -> Mouser
Changed lines of the file:
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@@
+      (effects (font (size 1.27 1.27)) hide)
+    )
+    (property "LCSC" "C107040" (id 8) (at 171.45 137.16 0)
       (effects (font (size 1.27 1.27)) hide)
     )
@@
     )
     (property "Distributor" "Mouser" (id 7) (at 156.21 137.16 0)
+      (effects (font (size 1.27 1.27)) hide)
+    )
+    (property "LCSC" "C107040" (id 8) (at 156.21 137.16 0)
       (effects (font (size 1.27 1.27)) hide)
     )
@@
       (effects (font (size 1.27 1.27)) hide)
     )
-    (property "Distributor" "" (id 7) (at 191.77 73.66 0)
+    (property "Distributor" "Mouser" (id 7) (at 191.77 73.66 0)
       (effects (font (size 1.27 1.27)) hide)
     )
@@
       (effects (font (size 1.27 1.27)) hide)
     )
+    (property "Checked" "y" (id 4) (at 233.68 118.11 0)
+      (effects (font (size 1.27 1.27)) hide)
+    )
+    (property "Distributor" "LCSC" (id 5) (at 233.68 118.11 0)
+      (effects (font (size 1.27 1.27)) hide)
+    )
+    (property "LCSC" "C165948" (id 6) (at 233.68 118.11 0)
+      (effects (font (size 1.27 1.27)) hide)
+    )
+    (property "Manufacturer" "Korean Hroparts" (id 7) (at 233.68 118.11 0)
+      (effects (font (size 1.27 1.27)) hide)
+    )
+    (property "Manufacturer_No" "TYPE-C-31-M-12" (id 8) (at 233.68 118.11 0)
+      (effects (font (size 1.27 1.27)) hide)
+    )
