File: reform2-motherboard25-pcb/reform2-pcie.kicad_sch (KiCad schematic)
At the start: 51 parts, among them J10 1-2199230-6, J11 48099-5701, U11 679105700, U20 AP22815, U23 IDT5V41066, Y3 25MHz

Commit message: motherboard 2.5 snapshot: fully routed and cleaned up
Parts:
- C119, C53, C54, C55, C59, C60, C61, R196: Distributor Mouser -> (none)
Changed lines of the file:
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@@
       (effects (font (size 1.27 1.27)) hide)
     )
-    (property "Distributor" "Mouser" (id 7) (at 138.43 48.26 0)
+    (property "Distributor" "" (id 7) (at 138.43 48.26 0)
       (effects (font (size 1.27 1.27)) hide)
     )
@@
       (effects (font (size 1.27 1.27)) hide)
     )
-    (property "Distributor" "Mouser" (id 7) (at 77.47 35.56 0)
+    (property "Distributor" "" (id 7) (at 77.47 35.56 0)
       (effects (font (size 1.27 1.27)) hide)
     )
@@
       (effects (font (size 1.27 1.27)) hide)
     )
-    (property "Distributor" "Mouser" (id 7) (at 87.63 35.56 0)
+    (property "Distributor" "" (id 7) (at 87.63 35.56 0)
       (effects (font (size 1.27 1.27)) hide)
     )
@@
       (effects (font (size 1.27 1.27)) hide)
     )
-    (property "Distributor" "Mouser" (id 7) (at 97.79 35.56 0)
+    (property "Distributor" "" (id 7) (at 97.79 35.56 0)
       (effects (font (size 1.27 1.27)) hide)
     )
@@
       (effects (font (size 1.27 1.27)) hide)
     )
-    (property "Distributor" "Mouser" (id 7) (at 203.2 40.64 0)
+    (property "Distributor" "" (id 7) (at 203.2 40.64 0)
       (effects (font (size 1.27 1.27)) hide)
     )
@@
       (effects (font (size 1.27 1.27)) hide)
     )
-    (property "Distributor" "Mouser" (id 7) (at 213.36 40.64 0)
+    (property "Distributor" "" (id 7) (at 213.36 40.64 0)
       (effects (font (size 1.27 1.27)) hide)
     )
@@
       (effects (font (size 1.27 1.27)) hide)
     )
-    (property "Distributor" "Mouser" (id 7) (at 223.52 40.64 0)
+    (property "Distributor" "" (id 7) (at 223.52 40.64 0)
       (effects (font (size 1.27 1.27)) hide)
     )
@@
       (effects (font (size 1.27 1.27)) hide)
     )
-    (property "Distributor" "Mouser" (id 7) (at 35.56 27.94 0)
-      (effects (font (size 1.27 1.27)) hide)
-    )
+    (property "Distributor" "" (id 7) (at 35.56 27.94 0)
+      (effects (font (size 1.27 1.27)) hide)
+    )

Commit message: motherboard25: r-1 snapshot, ordered for test bringup
Parts:
- C62, C98: LCSC (none) -> C107040
- R196: Distributor (none) -> Mouser
Changed lines of the file:
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@@
+      (effects (font (size 1.27 1.27)) hide)
+    )
+    (property "LCSC" "C107040" (id 8) (at 111.76 181.61 0)
       (effects (font (size 1.27 1.27)) hide)
     )
@@
     )
     (property "Distributor" "Mouser" (id 7) (at 96.52 181.61 0)
+      (effects (font (size 1.27 1.27)) hide)
+    )
+    (property "LCSC" "C107040" (id 8) (at 96.52 181.61 0)
       (effects (font (size 1.27 1.27)) hide)
     )
@@
       (effects (font (size 1.27 1.27)) hide)
     )
-    (property "Distributor" "" (id 7) (at 35.56 27.94 0)
-      (effects (font (size 1.27 1.27)) hide)
-    )
+    (property "Distributor" "Mouser" (id 7) (at 35.56 27.94 0)
+      (effects (font (size 1.27 1.27)) hide)
+    )
