File: reform2-motherboard25-pcb/reform2-power.kicad_sch (KiCad schematic)
At the start: 115 parts, among them J1 Jack-DC, J13 BATCON1, J2 BATCON2, Q1 Si7850DP, Q10 PMV50EPEAR, Q11 PMV50EPEAR, Q12 PMV50EPEAR, Q15 Si7850DP, Q17 Si7850DP, Q18 Si7461DP, Q2 Si7850DP, Q3 Si7461DP, Q4 PMV50ENEAR, Q5 PMV50EPEAR, Q6 PMV50EPEAR, Q7 PMV50EPEAR, Q8 PMV50EPEAR, Q9 PMV50EPEAR, U2 LTC4020EUHFPBF, U4 LTC6803-4, U6 PAC1921

Commit message: motherboard 2.5 snapshot: fully routed and cleaned up
Parts:
- C149, C2, C7, C80, R172, R54, R95: Distributor Mouser -> (none)
Changed lines of the file:
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@@
       (effects (font (size 1.27 1.27)) hide)
     )
-    (property "Distributor" "Mouser" (id 7) (at 149.86 82.55 0)
+    (property "Distributor" "" (id 7) (at 149.86 82.55 0)
       (effects (font (size 1.27 1.27)) hide)
     )
@@
       (effects (font (size 1.27 1.27)) hide)
     )
-    (property "Distributor" "Mouser" (id 7) (at 104.14 -25.4 0)
+    (property "Distributor" "" (id 7) (at 104.14 -25.4 0)
       (effects (font (size 1.27 1.27)) hide)
     )
@@
       (effects (font (size 1.27 1.27)) hide)
     )
-    (property "Distributor" "Mouser" (id 7) (at 86.36 40.64 0)
+    (property "Distributor" "" (id 7) (at 86.36 40.64 0)
       (effects (font (size 1.27 1.27)) hide)
     )
@@
       (effects (font (size 1.27 1.27)) hide)
     )
-    (property "Distributor" "Mouser" (id 5) (at 57.15 190.5 0)
+    (property "Distributor" "" (id 5) (at 57.15 190.5 0)
       (effects (font (size 1.27 1.27)) hide)
     )
@@
       (effects (font (size 1.27 1.27)) hide)
     )
-    (property "Distributor" "Mouser" (id 7) (at 36.83 176.53 0)
+    (property "Distributor" "" (id 7) (at 36.83 176.53 0)
       (effects (font (size 1.27 1.27)) hide)
     )
@@
       (effects (font (size 1.27 1.27)) hide)
     )
-    (property "Distributor" "Mouser" (id 5) (at 101.6 128.27 0)
+    (property "Distributor" "" (id 5) (at 101.6 128.27 0)
       (effects (font (size 1.27 1.27)) hide)
     )
@@
       (effects (font (size 1.27 1.27)) hide)
     )
-    (property "Distributor" "Mouser" (id 7) (at 95.25 168.91 0)
-      (effects (font (size 1.27 1.27)) hide)
-    )
+    (property "Distributor" "" (id 7) (at 95.25 168.91 0)
+      (effects (font (size 1.27 1.27)) hide)
+    )

Commit message: motherboard25: r-1 snapshot, ordered for test bringup
Parts:
- added R86: 100k, Resistor_SMD:R_0603_1608Metric, symbol Device:R_Small
- added R87: 10k, Resistor_SMD:R_0603_1608Metric, symbol Device:R_Small
- added R88, R89: 0, Resistor_SMD:R_0603_1608Metric, symbol Device:R_Small
- D17, D18, D19, D24, D25, D26, D27, D28: Checked (none) -> y; Distributor (none) -> Mouser; Manufacturer (none) -> Nexperia; Manufacturer_No (none) -> PMEG60T10ELRX
- R172, R54, R95: Distributor (none) -> Mouser
- R79: value 0 -> 100k NTC; symbol Device:R_Small -> Device:Thermistor_NTC; Manufacturer Vishay Dale -> Vishay / BC; Manufacturer_No CRCW06030000Z0EAC -> NTCS0603E3104FXT
- U2: Field4 ltc4020euhf#pbf -> (none)
- U6: Checked (none) -> y; Distributor (none) -> Mouser; Manufacturer (none) -> Microchip / Atmel; Manufacturer_No (none) -> PAC1921-1-AIA-TR
Connections:
- net GND: now also R88.1
- net LPC_VCC: now also R87.2, R89.2
- net at R79.1, U4.29 (Vtemp1): now also R86.1
- net at C4.1, U4.31 (Vref): now also R86.2
- net at U6.6 (ADDR_SEL): now also R88.2
- net at U6.7 (RESERVED): now also R89.1
- net at U6.8 (~{READ}/INT): now also R87.1
- no-connect marks 7 -> 6
Other:
- note added: "0R = I2C ADDR 1001_100"
- note added: "TODO: verify higher R on LEDs"
- note removed: "TODO: NTCs on the LTC6803-4"
- note removed: "TODO: double check with datasheet/ref circuit"
- note removed: "TODO: verify higher R"
- moved on the sheet: R78
