File: reform2-motherboard25-pcb/reform2-regulators.kicad_sch (KiCad schematic)
At the start: 53 parts, among them U12 LM2677SX-3.3, U13 TLV62568DBV, U14 LMR16006YQ3, U17 TLV1117-18, U19 TLV62568DBV, U7 LM2677SX-5

Commit message: motherboard25: r-1 snapshot, ordered for test bringup
Parts:
- D15, D16: Checked (none) -> y; Distributor (none) -> Mouser; Manufacturer (none) -> Vishay; Manufacturer_No (none) -> BZX584C3V3-G3-08
- R1: Manufacturer Vishay Dale -> Yageo; Manufacturer_No CRCW06030000Z0EAC -> RC0603FR-071ML
- R53, R57: Manufacturer Vishay Dale -> Yageo; Manufacturer_No CRCW0603100KJNEAC -> RC0603FR-0751KL
Changed lines of the file:
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@@
       (effects (font (size 1.27 1.27)) hide)
     )
-    (property "Manufacturer" "Vishay Dale" (id 4) (at 184.15 54.61 0)
-      (effects (font (size 1.27 1.27)) hide)
-    )
-    (property "Manufacturer_No" "CRCW06030000Z0EAC" (id 5) (at 184.15 54.61 0)
+    (property "Manufacturer" "Yageo" (id 4) (at 184.15 54.61 0)
+      (effects (font (size 1.27 1.27)) hide)
+    )
+    (property "Manufacturer_No" "RC0603FR-071ML" (id 5) (at 184.15 54.61 0)
       (effects (font (size 1.27 1.27)) hide)
     )
@@
       (effects (font (size 1.27 1.27)) hide)
     )
-    (property "Manufacturer" "Vishay Dale" (id 4) (at 81.28 52.07 0)
-      (effects (font (size 1.27 1.27)) hide)
-    )
-    (property "Manufacturer_No" "CRCW0603100KJNEAC" (id 5) (at 81.28 52.07 0)
+    (property "Manufacturer" "Yageo" (id 4) (at 81.28 52.07 0)
+      (effects (font (size 1.27 1.27)) hide)
+    )
+    (property "Manufacturer_No" "RC0603FR-0751KL" (id 5) (at 81.28 52.07 0)
       (effects (font (size 1.27 1.27)) hide)
     )
@@
       (effects (font (size 1.27 1.27)) hide)
     )
-    (property "Manufacturer" "Vishay Dale" (id 4) (at 81.28 87.63 0)
-      (effects (font (size 1.27 1.27)) hide)
-    )
-    (property "Manufacturer_No" "CRCW0603100KJNEAC" (id 5) (at 81.28 87.63 0)
+    (property "Manufacturer" "Yageo" (id 4) (at 81.28 87.63 0)
+      (effects (font (size 1.27 1.27)) hide)
+    )
+    (property "Manufacturer_No" "RC0603FR-0751KL" (id 5) (at 81.28 87.63 0)
       (effects (font (size 1.27 1.27)) hide)
     )
@@
       (effects (font (size 1.27 1.27)) hide)
     )
+    (property "Checked" "y" (id 4) (at 74.93 53.34 0)
+      (effects (font (size 1.27 1.27)) hide)
+    )
+    (property "Distributor" "Mouser" (id 5) (at 74.93 53.34 0)
+      (effects (font (size 1.27 1.27)) hide)
+    )
+    (property "Manufacturer" "Vishay" (id 6) (at 74.93 53.34 0)
+      (effects (font (size 1.27 1.27)) hide)
+    )
+    (property "Manufacturer_No" "BZX584C3V3-G3-08" (id 7) (at 74.93 53.34 0)
+      (effects (font (size 1.27 1.27)) hide)
+    )
     (pin "1")
     (pin "2")
@@
       (effects (font (size 1.27 1.27)) hide)
     )
+    (property "Checked" "y" (id 4) (at 74.93 88.9 0)
+      (effects (font (size 1.27 1.27)) hide)
+    )
+    (property "Distributor" "Mouser" (id 5) (at 74.93 88.9 0)
+      (effects (font (size 1.27 1.27)) hide)
+    )
+    (property "Manufacturer" "Vishay" (id 6) (at 74.93 88.9 0)
+      (effects (font (size 1.27 1.27)) hide)
+    )
+    (property "Manufacturer_No" "BZX584C3V3-G3-08" (id 7) (at 74.93 88.9 0)
+      (effects (font (size 1.27 1.27)) hide)
+    )
