File: reform2-motherboard25-pcb/reform2-usbpwr.kicad_sch (KiCad schematic)
At the start: 6 parts, among them U24 AP22815, U27 AP22815

Commit message: motherboard 2.5 snapshot: fully routed and cleaned up
Parts:
- R2, R83: Distributor Mouser -> (none)
Changed lines of the file:
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@@
       (effects (font (size 1.27 1.27)) hide)
     )
-    (property "Distributor" "Mouser" (id 7) (at 127 60.96 0)
+    (property "Distributor" "" (id 7) (at 127 60.96 0)
       (effects (font (size 1.27 1.27)) hide)
     )
@@
       (effects (font (size 1.27 1.27)) hide)
     )
-    (property "Distributor" "Mouser" (id 7) (at 67.31 60.96 0)
+    (property "Distributor" "" (id 7) (at 67.31 60.96 0)
       (effects (font (size 1.27 1.27)) hide)
     )

Commit message: motherboard25: r-1 snapshot, ordered for test bringup
Parts:
- R2, R83: Distributor (none) -> Mouser
Changed lines of the file:
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@@
       (effects (font (size 1.27 1.27)) hide)
     )
-    (property "Distributor" "" (id 7) (at 127 60.96 0)
+    (property "Distributor" "Mouser" (id 7) (at 127 60.96 0)
       (effects (font (size 1.27 1.27)) hide)
     )
@@
       (effects (font (size 1.27 1.27)) hide)
     )
-    (property "Distributor" "" (id 7) (at 67.31 60.96 0)
+    (property "Distributor" "Mouser" (id 7) (at 67.31 60.96 0)
       (effects (font (size 1.27 1.27)) hide)
     )
