File: reform2-keyboard3-pcb/reform2-keyboard3.kicad_sch (KiCad schematic)
At the start: 160 parts, among them SW1 Choc, SW10 Choc, SW11 Choc, SW12 Choc, SW13 Choc, SW14 Choc, SW15 Choc, SW16 Choc, SW17 Choc, SW18 Choc, SW19 Choc, SW2 Choc, SW20 Choc, SW21 Choc, SW22 Choc, SW23 Choc, SW24 Choc, SW25 Choc, SW26 Choc, SW27 Choc, SW28 Choc, SW29 Choc, SW3 Choc, SW30 Choc, SW31 Choc, SW32 Choc, SW33 Choc, SW34 Choc, SW35 Choc, SW37 Choc, SW38 Choc, SW39 Choc, SW4 Choc, SW40 Choc, SW41 Choc, SW42 Choc, SW43 Choc, SW44 Choc, SW45 Choc, SW46 Choc, SW47 Choc, SW48 Choc, SW49 Choc, SW5 Choc, SW50 Choc, SW51 Choc, SW52 Choc, SW53 Choc, SW54 Choc, SW55 Choc, SW56 Choc, SW57 Choc, SW58 Choc, SW59 Choc, SW6 Choc, SW60 Choc, SW61 Choc, SW62 Choc, SW63 Choc, SW64 Choc, SW65 Choc, SW66 Choc, SW67 Choc, SW68 Choc, SW69 Choc, SW7 Choc, SW70 Choc, SW71 Choc, SW72 Choc, SW73 Choc, SW74 Choc, SW75 Choc, SW76 Choc, SW77 Choc, SW78 Choc, SW79 Choc, SW8 Choc, SW80 Choc, SW82 Choc, SW9 Choc

Commit message: reform2-keyboard3: bump date, revision
Other:
- company: Copyright 2017-2020 MNT Research GmbH -> Copyright 2017-2023 MNT Research GmbH
Changed lines of the file:
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@@
   (title_block
     (title "MNT Reform 2 Keyboard")
-    (date "2022-03-03")
-    (rev "2.0R-2")
-    (company "Copyright 2017-2020 MNT Research GmbH")
+    (date "2023-01-17")
+    (rev "2.0R-3")
+    (company "Copyright 2017-2023 MNT Research GmbH")
     (comment 1 "https://mntre.com")
     (comment 2 "Engineer: Lukas F. Hartmann")
